Commit message: [rrbot] reduce the damping and unbalance the second link
- Reduce damping so arm swings as a double pendulum
- Offset the second link so the arm falls

File: ros_gz_sim_demos/models/rrbot.xacro (robot description, xacro)
@@ -52,5 +52,5 @@
     <origin xyz="0 ${width} ${height1 - axel_offset}" rpy="0 0 0"/>
     <axis xyz="0 1 0"/>
-    <dynamics damping="0.7"/>
+    <dynamics damping="0.01"/>
   </joint>
   <!-- Middle Link -->
@@ -83,5 +83,5 @@
     <origin xyz="0 ${width} ${height2 - axel_offset*2}" rpy="0 0 0"/>
     <axis xyz="0 1 0"/>
-    <dynamics damping="0.7"/>
+    <dynamics damping="0.01"/>
   </joint>
   <!-- Top Link -->
@@ -101,5 +101,5 @@
     </visual>
     <inertial>
-      <origin xyz="0 0 ${height3/2 - axel_offset}" rpy="0 0 0"/>
+      <origin xyz="0.01 0 ${height3/2 - axel_offset}" rpy="0 0 0"/>
       <mass value="${mass}"/>
       <inertia
